Commit message: Se creo una carpeta para cada robot dentro de quadruped_description, se añadio el archivo launch en formato xml

File: quadruped_description/Notspot/urdf/quadruped_robot.urdf (robot description, URDF)
Before this commit: robot quadruped, 17 links, 16 joints
Links:
- link FL1: geometry visual mesh filename=package://quadruped_description/Notspot/meshes/FL1_obj.obj
- link FL2: geometry collision cylinder length=0.125 radius=0.014; visual mesh filename=package://quadruped_description/Notspot/meshes/L2_obj.obj
- link FL3: geometry collision cylinder length=0.06 radius=0.007; visual mesh filename=package://quadruped_description/Notspot/meshes/L3_obj.obj
- link FR1: geometry visual mesh filename=package://quadruped_description/Notspot/meshes/FR1_obj.obj
- link FR2: geometry collision cylinder length=0.125 radius=0.014; visual mesh filename=package://quadruped_description/Notspot/meshes/R2_obj.obj
- link FR3: geometry collision cylinder length=0.06 radius=0.007; visual mesh filename=package://quadruped_description/Notspot/meshes/R3_obj.obj
- link RL1: geometry visual mesh filename=package://quadruped_description/Notspot/meshes/RL1_obj.obj
- link RL2: geometry collision cylinder length=0.125 radius=0.014; visual mesh filename=package://quadruped_description/Notspot/meshes/L2_obj.obj
- link RL3: geometry collision cylinder length=0.06 radius=0.007; visual mesh filename=package://quadruped_description/Notspot/meshes/L3_obj.obj
- link RR1: geometry visual mesh filename=package://quadruped_description/Notspot/meshes/RR1_obj.obj
- link RR2: geometry collision cylinder length=0.125 radius=0.014; visual mesh filename=package://quadruped_description/Notspot/meshes/R2_obj.obj
- link RR3: geometry collision cylinder length=0.06 radius=0.007; visual mesh filename=package://quadruped_description/Notspot/meshes/R3_obj.obj
- link base_link: geometry collision box size=0.25 0.1285 0.055; visual mesh filename=package://quadruped_description/Notspot/meshes/body_obj.obj
